Commit message: Update Mechabot description

File: urdf/mechabot_sensors.xacro (robot description, xacro)
@@ -11,4 +11,12 @@
             </material>
         </visual>
+        collision>
+            <origin xyz="-0.028 0.0 -0.132" rpy="0.0 0.0 0.0"/>
+            <geometry>
+                <mesh filename="package://mechabot_description/meshes/mechabot_lidar.stl" scale="0.001 0.001 0.001"/>
+            </geometry>
+            <material name="yellow">
+                <color rgba="0.5 0.5 0.0 1.0"/>
+            </material>
     </link>
     <joint name="lidar_joint" type="fixed">
@@ -27,4 +35,12 @@
             </material>
         </visual>
+        collision>
+            <origin xyz="-0.118 0.0 -0.092" rpy="0.0 0.0 0.0"/>
+            <geometry>
+                <mesh filename="package://mechabot_description/meshes/mechabot_camera.stl" scale="0.001 0.001 0.001"/>
+            </geometry>
+            <material name="yellow">
+                <color rgba="0.0 0.5 0.0 1.0"/>
+            </material>
     </link>
     <joint name="camera_joint" type="fixed">
@@ -43,4 +59,13 @@
             </material>
         </visual>
+        <collision>
+            <origin xyz="0.0 0.0 -0.035" rpy="0.0 0.0 0.0"/>
+            <geometry>
+                <mesh filename="package://mechabot_description/meshes/mechabot_imu.stl" scale="0.001 0.001 0.001"/>
+            </geometry>
+            <material name="yellow">
+                <color rgba="0.0 0.5 0.0 1.0"/>
+            </material>
+        </collision>
     </link>
     <joint name="imu_joint" type="fixed">
