Commit message: Update Mechabot robot description

File: urdf/mechabot.urdf.xacro (robot description, xacro)
@@ -3,3 +3,5 @@
     <xacro:include filename="$(find mechabot_description)/urdf/mechabot_base.xacro" />
     <xacro:include filename="$(find mechabot_description)/urdf/mechabot_sensors.xacro"/>
+    <xacro:include filename="$(find mechabot_description)/urdf/mechabot_gazebo.xacro"/>
+    <xacro:include filename="$(find mechabot_description)/urdf/mechabot_ros2control.xacro"/>
 </robot>

File: urdf/mechabot_base.xacro (robot description, xacro)
@@ -3,4 +3,9 @@
     <link name="base_footprint"/>
     <link name="base_link">
+       <inertial>
+            <origin xyz="0.0 0.0 -0.0125" rpy="0.0 0.0 0.0"/>
+            <mass value="5.0"/>
+            <inertia ixx="0.001" ixy="0.0" ixz="0.0" iyy="0.001" iyz="0.0" izz="0.001"/>
+       </inertial>
         <visual>
             <origin xyz="0.0 0.0 -0.0125" rpy="0.0 0.0 0.0"/>
@@ -28,6 +33,11 @@
     </joint>
     <link name="right_wheel_link">
-        <visual>
+        <inertial>
             <origin xyz="0.0 0.0925 -0.034" rpy="0.0 0.0 0.0"/>
+            <mass value="0.5"/>
+            <inertia ixx="0.001" ixy="0.0" ixz="0.0" iyy="0.001" iyz="0.0" izz="0.001"/>
+       </inertial>
+        <visual>
+            <origin xyz="0.0 0.0925 -0.034" rpy="0.0 0.0 0.0"/>
             <geometry>
                 <mesh filename="package://mechabot_description/meshes/mechabot_right_wheel.stl" scale="0.001 0.001 0.001"/>
@@ -38,7 +48,8 @@
         </visual>
         <collision>
-            <origin xyz="0.0 0.0925 -0.034" rpy="0.0 0.0 0.0"/>
-            <geometry>
-                <mesh filename="package://mechabot_description/meshes/mechabot_right_wheel.stl" scale="0.001 0.001 0.001"/>
+            <origin xyz="0.0 0.0 0.0" rpy="0.0 0.0 0.0"/>
+            <geometry>
+                <sphere radius="0.034"/>
+                <!-- <mesh filename="package://mechabot_description/meshes/mechabot_right_wheel.stl" scale="0.001 0.001 0.001"/> -->
             </geometry>
             <material name="blue">
@@ -54,6 +65,11 @@
     </joint>
     <link name="left_wheel_link">
-        <visual>
+        <inertial>
             <origin xyz="0.0 -0.0925 -0.034" rpy="0.0 0.0 0.0"/>
+            <mass value="0.5"/>
+            <inertia ixx="0.001" ixy="0.0" ixz="0.0" iyy="0.001" iyz="0.0" izz="0.001"/>
+        </inertial>
+        <visual>
+            <origin xyz="0.0 -0.0925 -0.034" rpy="0.0 0.0 0.0"/>
             <geometry>
                 <mesh filename="package://mechabot_description/meshes/mechabot_left_wheel.stl" scale="0.001 0.001 0.001"/>
@@ -64,7 +80,8 @@
         </visual>
         <collision>
-            <origin xyz="0.0 -0.0925 -0.034" rpy="0.0 0.0 0.0"/>
-            <geometry>
-                <mesh filename="package://mechabot_description/meshes/mechabot_left_wheel.stl" scale="0.001 0.001 0.001"/>
+            <origin xyz="0.0 0.0 0.0" rpy="0.0 0.0 0.0"/>
+            <geometry>
+                <sphere radius="0.034"/>
+                <!-- <mesh filename="package://mechabot_description/meshes/mechabot_left_wheel.stl" scale="0.001 0.001 0.001"/> -->
             </geometry>
             <material name="blue">
@@ -80,6 +97,11 @@
     </joint>
     <link name="front_left_castor_link">
-        <visual>
+        <inertial>
             <origin xyz="-0.085 -0.065 -0.021" rpy="0.0 0.0 0.0"/>
+            <mass value="0.2"/>
+            <inertia ixx="0.001" ixy="0.0" ixz="0.0" iyy="0.001" iyz="0.0" izz="0.001"/>
+        </inertial>
+        <visual>
+            <origin xyz="-0.085 -0.065 -0.021" rpy="0.0 0.0 0.0"/>
             <geometry>
                 <mesh filename="package://mechabot_description/meshes/front_left_castor.stl" scale="0.001 0.001 0.001"/>
@@ -90,7 +112,8 @@
         </visual>
         <collision>
-            <origin xyz="-0.085 -0.065 -0.021" rpy="0.0 0.0 0.0"/>
-            <geometry>
-                <mesh filename="package://mechabot_description/meshes/front_left_castor.stl" scale="0.001 0.001 0.001"/>
+            <origin xyz="0.0 0.0 0.0" rpy="0.0 0.0 0.0"/>
+            <geometry>
+                <sphere radius="0.00625"/>
+                <!-- <mesh filename="package://mechabot_description/meshes/front_left_castor.stl" scale="0.001 0.001 0.001"/> -->
             </geometry>
             <material name="grey">
@@ -105,6 +128,11 @@
     </joint>
     <link name="front_right_castor_link">
-        <visual>
+        <inertial>
             <origin xyz="-0.085 0.065 -0.021" rpy="0.0 0.0 0.0"/>
+            <mass value="0.2"/>
+            <inertia ixx="0.001" ixy="0.0" ixz="0.0" iyy="0.001" iyz="0.0" izz="0.001"/>
+        </inertial>
+        <visual>
+            <origin xyz="-0.085 0.065 -0.021" rpy="0.0 0.0 0.0"/>
             <geometry>
                 <mesh filename="package://mechabot_description/meshes/front_right_castor.stl" scale="0.001 0.001 0.001"/>
@@ -115,7 +143,8 @@
         </visual>
         <collision>
-            <origin xyz="-0.085 0.065 -0.021" rpy="0.0 0.0 0.0"/>
-            <geometry>
-                <mesh filename="package://mechabot_description/meshes/front_right_castor.stl" scale="0.001 0.001 0.001"/>
+            <origin xyz="0.0 0.0 0.0" rpy="0.0 0.0 0.0"/>
+            <geometry>
+                <sphere radius="0.00625"/>
+                <!-- <mesh filename="package://mechabot_description/meshes/front_right_castor.stl" scale="0.001 0.001 0.001"/> -->
             </geometry>
             <material name="grey">
@@ -130,6 +159,11 @@
     </joint>
     <link name="rear_left_castor_link">
-        <visual>
+        <inertial>
             <origin xyz="0.085 -0.065 -0.0205" rpy="0.0 0.0 0.0"/>
+            <mass value="0.2"/>
+            <inertia ixx="0.001" ixy="0.0" ixz="0.0" iyy="0.001" iyz="0.0" izz="0.001"/>
+        </inertial>
+        <visual>
+            <origin xyz="0.085 -0.065 -0.0205" rpy="0.0 0.0 0.0"/>
             <geometry>
                 <mesh filename="package://mechabot_description/meshes/rear_left_castor.stl" scale="0.001 0.001 0.001"/>
@@ -140,7 +174,8 @@
         </visual>
         <collision>
-            <origin xyz="0.085 -0.065 -0.0205" rpy="0.0 0.0 0.0"/>
-            <geometry>
-                <mesh filename="package://mechabot_description/meshes/rear_left_castor.stl" scale="0.001 0.001 0.001"/>
+            <origin xyz="0.0 0.0 0.0" rpy="0.0 0.0 0.0"/>
+            <geometry>
+                <sphere radius="0.00625"/>
+                <!-- <mesh filename="package://mechabot_description/meshes/rear_left_castor.stl" scale="0.001 0.001 0.001"/> -->
             </geometry>
             <material name="grey">
@@ -155,6 +190,11 @@
     </joint>
     <link name="rear_right_castor_link">
-        <visual>
+        <inertial>
             <origin xyz="0.085 0.065 -0.0205" rpy="0.0 0.0 0.0"/>
+            <mass value="0.2"/>
+            <inertia ixx="0.001" ixy="0.0" ixz="0.0" iyy="0.001" iyz="0.0" izz="0.001"/>
+        </inertial>
+        <visual>
+            <origin xyz="0.085 0.065 -0.0205" rpy="0.0 0.0 0.0"/>
             <geometry>
                 <mesh filename="package://mechabot_description/meshes/rear_right_castor.stl" scale="0.001 0.001 0.001"/>
@@ -165,7 +205,8 @@
         </visual>
         <collision>
-            <origin xyz="0.085 0.065 -0.0205" rpy="0.0 0.0 0.0"/>
-            <geometry>
-                <mesh filename="package://mechabot_description/meshes/rear_right_castor.stl" scale="0.001 0.001 0.001"/>
+            <origin xyz="0.0 0.0 0.0" rpy="0.0 0.0 0.0"/>
+            <geometry>
+                <sphere radius="0.00625"/>
+                <!-- <mesh filename="package://mechabot_description/meshes/rear_right_castor.stl" scale="0.001 0.001 0.001"/> -->
             </geometry>
             <material name="grey">
@@ -180,4 +221,9 @@
     </joint>
     <link name="toplid_link">
+        <inertial>
+            <origin xyz="0.0 0.0 -0.001125" rpy="0.0 0.0 0.0"/>
+            <mass value="2.0"/>
+            <inertia ixx="0.001" ixy="0.0" ixz="0.0" iyy="0.001" iyz="0.0" izz="0.001"/>
+        </inertial>
         <visual>
             <origin xyz="0.0 0.0 -0.1125" rpy="0.0 0.0 0.0"/>

File: urdf/mechabot_sensors.xacro (robot description, xacro)
@@ -2,4 +2,9 @@
 <robot name="bot_name" xmlns:xacro="http://www.ros.org/wiki/xacro">
     <link name="lidar_link">
+        <inertial>
+            <origin xyz="-0.028 0.0 -0.132" rpy="0.0 0.0 0.0"/>
+            <mass value="0.5"/>
+            <inertia ixx="0.001" ixy="0.0" ixz="0.0" iyy="0.001" iyz="0.0" izz="0.001"/>
+        </inertial>
         <visual>
             <origin xyz="-0.028 0.0 -0.132" rpy="0.0 0.0 0.0"/>
@@ -11,5 +16,5 @@
             </material>
         </visual>
-        collision>
+        <collision>
             <origin xyz="-0.028 0.0 -0.132" rpy="0.0 0.0 0.0"/>
             <geometry>
@@ -19,4 +24,5 @@
                 <color rgba="0.5 0.5 0.0 1.0"/>
             </material>
+        </collision>
     </link>
     <joint name="lidar_joint" type="fixed">
@@ -26,4 +32,9 @@
     </joint>
      <link name="camera_link">
+        <inertial>
+            <origin xyz="-0.118 0.0 -0.092" rpy="0.0 0.0 0.0"/>
+            <mass value="0.1"/>
+            <inertia ixx="0.001" ixy="0.0" ixz="0.0" iyy="0.001" iyz="0.0" izz="0.001"/>
+        </inertial>
         <visual>
             <origin xyz="-0.118 0.0 -0.092" rpy="0.0 0.0 0.0"/>
@@ -35,5 +46,5 @@
             </material>
         </visual>
-        collision>
+        <collision>
             <origin xyz="-0.118 0.0 -0.092" rpy="0.0 0.0 0.0"/>
             <geometry>
@@ -43,4 +54,5 @@
                 <color rgba="0.0 0.5 0.0 1.0"/>
             </material>
+            </collision>
     </link>
     <joint name="camera_joint" type="fixed">
@@ -50,4 +62,9 @@
     </joint>
     <link name="imu_link">
+        <inertial>
+            <origin xyz="0.0 0.0 -0.035" rpy="0.0 0.0 0.0"/>
+            <mass value="0.1"/>
+            <inertia ixx="0.001" ixy="0.0" ixz="0.0" iyy="0.001" iyz="0.0" izz="0.001"/>
+        </inertial>
         <visual>
             <origin xyz="0.0 0.0 -0.035" rpy="0.0 0.0 0.0"/>
