Commit message: Add launch file and update robot description

File: urdf/mechabot_base.xacro (robot description, xacro)
@@ -29,8 +29,9 @@
         </visual>
     </link>
-    <joint name="right_wheel_joint" type="fixed">
+    <joint name="right_wheel_joint" type="continuous">
         <origin xyz="0.0 -0.0925 0.0215" rpy="0.0 0.0 0.0"/>
         <parent link="base_link"/>
         <child link="right_wheel_link"/>
+        <axis xyz="0 1 0"/>
     </joint>
     <link name="left_wheel_link">
@@ -45,8 +46,89 @@
         </visual>
     </link>
-    <joint name="left_wheel_joint" type="fixed">
+    <joint name="left_wheel_joint" type="continuous">
         <origin xyz="0.0 0.0925 0.0215" rpy="0.0 0.0 0.0"/>
         <parent link="base_link"/>
         <child link="left_wheel_link"/>
+        <axis xyz="0 1 0"/>
+    </joint>
+    <link name="front_left_castor_link">
+        <visual>
+            <origin xyz="-0.085 -0.065 -0.021" rpy="0.0 0.0 0.0"/>
+            <geometry>
+                <mesh filename="package://mechabot_description/meshes/front_left_castor.stl" scale="0.001 0.001 0.001"/>
+            </geometry>
+            <material name="grey">
+                <color rgba="0.6 0.6 0.6 1.0"/>
+            </material>
+        </visual>
+    </link>
+    <joint name="front_left_castor_joint" type="fixed">
+        <origin xyz="0.085 0.065 0.0085" rpy="0.0 0.0 0.0"/>
+        <parent link="base_link"/>
+        <child link="front_left_castor_link"/>
+    </joint>
+    <link name="front_right_castor_link">
+        <visual>
+            <origin xyz="-0.085 0.065 -0.021" rpy="0.0 0.0 0.0"/>
+            <geometry>
+                <mesh filename="package://mechabot_description/meshes/front_right_castor.stl" scale="0.001 0.001 0.001"/>
+            </geometry>
+            <material name="grey">
+                <color rgba="0.6 0.6 0.6 1.0"/>
+            </material>
+        </visual>
+    </link>
+    <joint name="front_right_castor_joint" type="fixed">
+        <origin xyz="0.085 -0.065 0.0085" rpy="0.0 0.0 0.0"/>
+        <parent link="base_link"/>
+        <child link="front_right_castor_link"/>
+    </joint>
+    <link name="rear_left_castor_link">
+        <visual>
+            <origin xyz="0.085 -0.065 -0.0205" rpy="0.0 0.0 0.0"/>
+            <geometry>
+                <mesh filename="package://mechabot_description/meshes/rear_left_castor.stl" scale="0.001 0.001 0.001"/>
+            </geometry>
+            <material name="grey">
+                <color rgba="0.6 0.6 0.6 1.0"/>
+            </material>
+        </visual>
+    </link>
+    <joint name="rear_left_castor_joint" type="fixed">
+        <origin xyz="-0.085 0.065 0.008" rpy="0.0 0.0 0.0"/>
+        <parent link="base_link"/>
+        <child link="rear_left_castor_link"/>
+    </joint>
+    <link name="rear_right_castor_link">
+        <visual>
+            <origin xyz="0.085 0.065 -0.0205" rpy="0.0 0.0 0.0"/>
+            <geometry>
+                <mesh filename="package://mechabot_description/meshes/rear_right_castor.stl" scale="0.001 0.001 0.001"/>
+            </geometry>
+            <material name="grey">
+                <color rgba="0.6 0.6 0.6 1.0"/>
+            </material>
+        </visual>
+    </link>
+    <joint name="rear_right_castor_joint" type="fixed">
+        <origin xyz="-0.085 -0.065 0.008" rpy="0.0 0.0 0.0"/>
+        <parent link="base_link"/>
+        <child link="rear_right_castor_link"/>
+    </joint>
+    <link name="toplid_link">
+        <visual>
+            <origin xyz="0.0 0.0 -0.1125" rpy="0.0 0.0 0.0"/>
+            <geometry>
+                <mesh filename="package://mechabot_description/meshes/mechabot_toplid.stl" scale="0.001 0.001 0.001"/>
+            </geometry>
+            <material name="red">
+                <color rgba="1.0 0.0 0.0 1.0"/>
+            </material>
+        </visual>
+    </link>
+    <joint name="toplid_joint" type="fixed">
+        <origin xyz="0.0 0.0 0.1" rpy="0.0 0.0 0.0"/>
+        <parent link="base_link"/>
+        <child link="toplid_link"/>
     </joint>
 </robot>

Commit message: Update collision geometry

File: urdf/mechabot_base.xacro (robot description, xacro)
@@ -12,4 +12,13 @@
             </material>
         </visual>
+        <collision>
+            <origin xyz="0.0 0.0 -0.0125" rpy="0.0 0.0 0.0"/>
+            <geometry>
+                <mesh filename="package://mechabot_description/meshes/mechabot_base_link.stl" scale="0.001 0.001 0.001"/> -->
+            </geometry>
+            <material name="grey">
+                <color rgba="0.5 0.5 0.5 1.0"/>
+            </material>
+        </collision>
     </link>
     <joint name="base_joint" type="fixed">
@@ -28,4 +37,13 @@
             </material>
         </visual>
+        <collision>
+            <origin xyz="0.0 0.0925 -0.034" rpy="0.0 0.0 0.0"/>
+            <geometry>
+                <mesh filename="package://mechabot_description/meshes/mechabot_right_wheel.stl" scale="0.001 0.001 0.001"/>
+            </geometry>
+            <material name="blue">
+                <color rgba="0.0 0.0 0.6 1.0"/>
+            </material>
+        </collision>
     </link>
     <joint name="right_wheel_joint" type="continuous">
@@ -45,4 +63,13 @@
             </material>
         </visual>
+        <collision>
+            <origin xyz="0.0 -0.0925 -0.034" rpy="0.0 0.0 0.0"/>
+            <geometry>
+                <mesh filename="package://mechabot_description/meshes/mechabot_left_wheel.stl" scale="0.001 0.001 0.001"/>
+            </geometry>
+            <material name="blue">
+                <color rgba="0.0 0.0 0.6 1.0"/>
+            </material>
+        </collision>
     </link>
     <joint name="left_wheel_joint" type="continuous">
@@ -62,4 +89,13 @@
             </material>
         </visual>
+        <collision>
+            <origin xyz="-0.085 -0.065 -0.021" rpy="0.0 0.0 0.0"/>
+            <geometry>
+                <mesh filename="package://mechabot_description/meshes/front_left_castor.stl" scale="0.001 0.001 0.001"/>
+            </geometry>
+            <material name="grey">
+                <color rgba="0.6 0.6 0.6 1.0"/>
+            </material>
+        </collision>
     </link>
     <joint name="front_left_castor_joint" type="fixed">
@@ -78,4 +114,13 @@
             </material>
         </visual>
+        <collision>
+            <origin xyz="-0.085 0.065 -0.021" rpy="0.0 0.0 0.0"/>
+            <geometry>
+                <mesh filename="package://mechabot_description/meshes/front_right_castor.stl" scale="0.001 0.001 0.001"/>
+            </geometry>
+            <material name="grey">
+                <color rgba="0.6 0.6 0.6 1.0"/>
+            </material>
+        </collision>
     </link>
     <joint name="front_right_castor_joint" type="fixed">
@@ -94,4 +139,13 @@
             </material>
         </visual>
+        <collision>
+            <origin xyz="0.085 -0.065 -0.0205" rpy="0.0 0.0 0.0"/>
+            <geometry>
+                <mesh filename="package://mechabot_description/meshes/rear_left_castor.stl" scale="0.001 0.001 0.001"/>
+            </geometry>
+            <material name="grey">
+                <color rgba="0.6 0.6 0.6 1.0"/>
+            </material>
+        </collision>
     </link>
     <joint name="rear_left_castor_joint" type="fixed">
@@ -110,4 +164,13 @@
             </material>
         </visual>
+        <collision>
+            <origin xyz="0.085 0.065 -0.0205" rpy="0.0 0.0 0.0"/>
+            <geometry>
+                <mesh filename="package://mechabot_description/meshes/rear_right_castor.stl" scale="0.001 0.001 0.001"/>
+            </geometry>
+            <material name="grey">
+                <color rgba="0.6 0.6 0.6 1.0"/>
+            </material>
+        </collision>
     </link>
     <joint name="rear_right_castor_joint" type="fixed">
@@ -126,4 +189,13 @@
             </material>
         </visual>
+        <collision>
+            <origin xyz="0.0 0.0 -0.1125" rpy="0.0 0.0 0.0"/>
+            <geometry>
+                <mesh filename="package://mechabot_description/meshes/mechabot_toplid.stl" scale="0.001 0.001 0.001"/>
+            </geometry>
+            <material name="red">
+                <color rgba="1.0 0.0 0.0 1.0"/>
+            </material>
+        </collision>
     </link>
     <joint name="toplid_joint" type="fixed">

Commit message: Update Mechabot description, Gazebo and ros2_control

File: urdf/mechabot_base.xacro (robot description, xacro)
@@ -112,5 +112,5 @@
         </visual>
         <collision>
-            <origin xyz="0.0 0.0 0.0" rpy="0.0 0.0 0.0"/>
+            <origin xyz="0.0 0.0 -0.0125" rpy="0.0 0.0 0.0"/>
             <geometry>
                 <sphere radius="0.00625"/>
@@ -123,5 +123,5 @@
     </link>
     <joint name="front_left_castor_joint" type="fixed">
-        <origin xyz="0.085 0.065 0.0085" rpy="0.0 0.0 0.0"/>
+        <origin xyz="0.085 0.065 0.00625" rpy="0.0 0.0 0.0"/>
         <parent link="base_link"/>
         <child link="front_left_castor_link"/>
@@ -143,5 +143,5 @@
         </visual>
         <collision>
-            <origin xyz="0.0 0.0 0.0" rpy="0.0 0.0 0.0"/>
+            <origin xyz="0.0 0.0 -0.0125" rpy="0.0 0.0 0.0"/>
             <geometry>
                 <sphere radius="0.00625"/>
@@ -154,5 +154,5 @@
     </link>
     <joint name="front_right_castor_joint" type="fixed">
-        <origin xyz="0.085 -0.065 0.0085" rpy="0.0 0.0 0.0"/>
+        <origin xyz="0.085 -0.065 0.00625" rpy="0.0 0.0 0.0"/>
         <parent link="base_link"/>
         <child link="front_right_castor_link"/>
@@ -174,5 +174,5 @@
         </visual>
         <collision>
-            <origin xyz="0.0 0.0 0.0" rpy="0.0 0.0 0.0"/>
+            <origin xyz="0.0 0.0 -0.0125" rpy="0.0 0.0 0.0"/>
             <geometry>
                 <sphere radius="0.00625"/>
@@ -185,5 +185,5 @@
     </link>
     <joint name="rear_left_castor_joint" type="fixed">
-        <origin xyz="-0.085 0.065 0.008" rpy="0.0 0.0 0.0"/>
+        <origin xyz="-0.085 0.065 0.00635" rpy="0.0 0.0 0.0"/>
         <parent link="base_link"/>
         <child link="rear_left_castor_link"/>
@@ -205,5 +205,5 @@
         </visual>
         <collision>
-            <origin xyz="0.0 0.0 0.0" rpy="0.0 0.0 0.0"/>
+            <origin xyz="0.0 0.0 -0.0125" rpy="0.0 0.0 0.0"/>
             <geometry>
                 <sphere radius="0.00625"/>
@@ -216,5 +216,5 @@
     </link>
     <joint name="rear_right_castor_joint" type="fixed">
-        <origin xyz="-0.085 -0.065 0.008" rpy="0.0 0.0 0.0"/>
+        <origin xyz="-0.085 -0.065 0.00635" rpy="0.0 0.0 0.0"/>
         <parent link="base_link"/>
         <child link="rear_right_castor_link"/>
